File: electronics/PIR.sch (EAGLE design)
At the start: 7 parts, among them X1 MAB5SV, X2 MAB3SH, X3 MAB5SV, X4 MAB5SV, X5 MAB5SV, X6 MAB5SV

Commit message: Added label indicator
Other:
- note added: "1"
Changed lines of the file:
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@@
 <sheet>
 <plain>
+<text x="182.88" y="63.5" size="5.08" layer="91">1</text>
 </plain>
 <instances>
